File: hardware/ESPHome_SHT4X/ESPHome_SHT4X.kicad_pcb (KiCad board)
At the start: 2 copper layers, 50 x 37.4 mm, 41 parts, among them J2 UJ20-C-H-G-SMT-2A-P16-TR, SW1 SW_Push, SW2 SW_Push, SW3 SW_Push, U1 ESP32-C6-WROOM-1-N8, U2 BQ25628ERYKR, U3 SHT40-AD1F-R2, U4 XC6220B331MR-G

Commit message: Making progress
Parts:
- added D3: LED, LED_SMD:LED_1206_3216Metric_Pad1.42x1.75mm_HandSolder, F.Cu at (150.0, 57.0)
- added R17: 1k, Resistor_SMD:R_01005_0402Metric_Pad0.57x0.30mm_HandSolder, F.Cu at (146.0, 57.0)
- C1, C10, C11, C12, C13, C14, C15, C16, C4, C5, C6, C7, C8, C9: footprint Capacitor_SMD:C_1206_3216Metric_Pad1.33x1.80mm_HandSolder -> Capacitor_SMD:C_01005_0402Metric_Pad0.57x0.30mm_HandSolder
- C2, C3: footprint LED_SMD:LED_Kingbright_APFA3010_3x1.5mm_Horizontal -> Capacitor_SMD:C_01005_0402Metric_Pad0.57x0.30mm_HandSolder
- L1: footprint Inductor_SMD:L_1206_3216Metric_Pad1.22x1.90mm_HandSolder -> Resistor_SMD:R_01005_0402Metric_Pad0.57x0.30mm_HandSolder
- R10, R13, R8: footprint Resistor_SMD:R_1206_3216Metric_Pad1.30x1.75mm_HandSolder -> Inductor_SMD:L_01005_0402Metric_Pad0.57x0.30mm_HandSolder
- R11, R12, R14, R15, R16, R3, R4, R5, R6, R7, R9: footprint Resistor_SMD:R_1206_3216Metric_Pad1.30x1.75mm_HandSolder -> Resistor_SMD:R_01005_0402Metric_Pad0.57x0.30mm_HandSolder
- moved J2 97.3 mm to (137.2, 50.0), turned to 180 degrees
- moved U4 95.7 mm to (134.2, 61.0), turned to -90 degrees
- moved D2 87.9 mm to (155.5, 59.9)
- moved D1 87.2 mm to (155.5, 57.3)
- moved U2 86.0 mm to (155.4, 63.4)
- moved R6 62.9 mm to (152.2, 63.4)
- moved SW3 61.5 mm to (173.8, 80.5)
- moved SW2 56.7 mm to (164.2, 80.5)
- moved R5 55.5 mm to (156.4, 66.3), turned to -90 degrees
- moved SW1 54.3 mm to (154.8, 80.5)
- moved U3 10.4 mm to (137.3, 80.4)
Routing:
- net SCL: track 0.00 -> 3.86 mm
- net ESP_3V3: track 0.00 -> 3.81 mm
- net GND: track 0.00 -> 3.16 mm
- net SDA: track 0.00 -> 3.14 mm
- net SYS: track 0.00 -> 2.75 mm
- added copper zone on F.Cu, net GND
Other:
- outline, holes or cut-outs redrawn
