File: hardware/ESPHome_SHT4X/ESPHome_SHT4X.kicad_pcb (KiCad board)
At the start: 2 copper layers, 43.4 x 30.5 mm, 45 parts, among them J2 UJ20-C-H-G-SMT-2A-P16-TR, U1 ESP32-C6-WROOM-1-N8, U2 BQ25628ERYKR, U3 SHT40-AD1F-R2, U4 XC6220B331MR-G

Commit message: Working
Parts:
- moved REF** 37.6 mm to (143.6, 82.7)
- moved R4 31.5 mm to (144.6, 66.7), turned to 180 degrees
- moved D3 31.3 mm to (180.3, 62.2)
- moved S1 31.3 mm to (178.3, 81.0), turned to 0 degrees
- moved R3 31.1 mm to (146.2, 65.9), turned to 180 degrees
- moved R17 28.7 mm to (177.2, 62.2), turned to -90 degrees
- moved J2 28.1 mm to (182.5, 68.8), turned to 90 degrees
- moved Jr1 26.6 mm to (156.8, 59.5), turned to 180 degrees
- moved R5 23.2 mm to (162.2, 61.5), turned to 180 degrees
- moved R7 20.9 mm to (175.6, 66.6), turned to 180 degrees
- moved C13 20.8 mm to (175.9, 69.7), turned to -90 degrees
- moved D1 20.5 mm to (161.8, 57.2), turned to 0 degrees
- moved D2 18.9 mm to (156.7, 62.7), turned to 0 degrees
- moved R10 18.6 mm to (174.6, 69.3), turned to 0 degrees
- moved C14 18.6 mm to (176.0, 67.9), turned to 90 degrees
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Connections:
- R14 pad 2: IO18 -> *CE
- U1 pad 16: IO18 -> SDA
- U1 pad 17: IO19 -> SCL
- U1 pad 18: IO20 -> *CE
- U1 pad 30_1: (no net) -> GND
- U1 pad 30_10: (no net) -> GND
- U1 pad 30_11: (no net) -> GND
- U1 pad 30_12: (no net) -> GND
- U1 pad 30_2: (no net) -> GND
- U1 pad 30_3: (no net) -> GND
- U1 pad 30_6: (no net) -> GND
- U1 pad 30_7: (no net) -> GND
- U1 pad 30_8: (no net) -> GND
- U1 pad 30_9: (no net) -> GND
- U1 pad 6: SDA -> unconnected-(U1-IO6-Pad6)
- U1 pad 7: SCL -> unconnected-(U1-IO7-Pad7)
- U1 pad r: (no net) -> GND
- U2 pad 14: IO18 -> *CE
Routing:
- net Net-(U2-*PG): track 30.5 -> 2.75 mm
- net *CE: track 0.00 -> 24.8 mm
- net SDA: track 58.5 -> 34.7 mm
- net *INT: track 8.83 -> 30.8 mm
- net SCL: track 55.9 -> 38.1 mm
- net EN: track 32.9 -> 15.4 mm, vias 1 -> 0
- net Net-(D2-K): track 1.80 -> 19.1 mm
- net GND: track 7.78 -> 24.4 mm, vias 21 -> 49
- net Net-(U1-IO12): track 16.9 -> 4.41 mm
- net Net-(U1-IO13): track 16.8 -> 4.49 mm
- net ESP_3V3: track 62.8 -> 74.7 mm, vias 0 -> 8
- net IO18: track 6.28 -> 0.00 mm, vias 1 -> 0
- net Net-(D1-K): track 0.68 -> 6.65 mm, vias 0 -> 2
- net VBUS: track 18.4 -> 23.2 mm
- net Net-(U2-STAT): track 0.00 -> 4.42 mm, vias 1 -> 2
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- added copper zone on F.Cu, net ESP_3V3

Commit message: Working
Parts:
- D1, D2, D3: footprint LED_SMD:LED_1206_3216Metric_Pad1.42x1.75mm_HandSolder -> LED_SMD:LED_0603_1608Metric_Pad1.05x0.95mm_HandSolder
- moved C1 4.32 mm to (143.5, 59.8), turned to -90 degrees
- moved C10 0.53 mm to (168.8, 56.5)
- moved D3 0.33 mm to (179.9, 62.1)
- moved C4 0.26 mm to (170.3, 58.2)
- moved D1 0.08 mm to (161.8, 57.1)
- moved D2 0.07 mm to (156.6, 62.7)
Connections:
- U1 pad 30_1: GND -> (no net)
- U1 pad 30_10: GND -> (no net)
- U1 pad 30_11: GND -> (no net)
- U1 pad 30_12: GND -> (no net)
- U1 pad 30_2: GND -> (no net)
- U1 pad 30_3: GND -> (no net)
- U1 pad 30_6: GND -> (no net)
- U1 pad 30_7: GND -> (no net)
- U1 pad 30_8: GND -> (no net)
- U1 pad 30_9: GND -> (no net)
- U1 pad gnd: GND -> (no net)
- U1 pad r: GND -> (no net)
Routing:
- net GND: track 24.4 -> 35.2 mm, vias 49 -> 154
- net BTST: track 0.99 -> 3.30 mm
- net SYS: track 12.7 -> 14.0 mm
- net Net-(D1-K): track 6.65 -> 7.29 mm
- net Net-(D2-K): track 19.1 -> 19.7 mm
- net SW: vias 10 -> 9
- added copper zone on F.Cu, net Net-(U2-STAT)
Other:
- board text added: "BOOT"
- board text added: "RESET"
