File: hardware/ESPHome_SHT4X/inputpower.kicad_sch (KiCad schematic)
At the start: 10 parts, among them J1 USB_C_Receptacle_USB2.0_14P, U3 SHT40-AD1F-R2, U4 XC6220B331MR-G

Commit message: Finishing touches on schematic, started on PCB Design
Parts:
- removed J1: USB_C_Receptacle_USB2.0_14P, RF_Module:ESP32-S2-WROVER, symbol Connector:USB_C_Receptacle_USB2.0_14P
- removed R1, R2: 5.1k, symbol Device:R_US
- added J2: UJ20-C-H-G-SMT-2A-P16-TR, Library:SAMESKY_UJ20-C-H-G-SMT-2A-P16-TR, symbol local:UJ20-C-H-G-SMT-2A-P16-TR
- added R16, R7: 5.1k, Resistor_SMD:R_1206_3216Metric_Pad1.30x1.75mm_HandSolder, symbol Device:R_US
- C1: footprint (none) -> Capacitor_SMD:C_1206_3216Metric_Pad1.33x1.80mm_HandSolder
- R3, R4: footprint (none) -> Resistor_SMD:R_1206_3216Metric_Pad1.30x1.75mm_HandSolder
- U3: footprint SHT40-AD1F-R2:SHT4X -> Library:SHT4X
- U4: footprint SOT-25_TOR -> Library:SOT-25_TOR
Connections:
- net +3.3V: now also C3.1
- net D+: now also J2.A6 (DP1), J2.A7 (DN1)
- net D-: now also J2.B6 (DP2), J2.B7 (DN2)
- net GND: now also C3.2, J2.A1_B12 (GND), J2.B1_A12 (GND__1), J2.SH1 (SHIELD), J2.SH2 (SHIELD__1), J2.SH3 (SHIELD__2), J2.SH4 (SHIELD__3), R16.2, R7.2; no longer U4.3 (CE)
- net SYS: now also U4.3 (CE)
- net VBUS: now also J2.A4_B9 (VBUS), J2.B4_A9 (VBUS__1)
- new net: J2.A5 (CC1), R16.1
- new net: J2.B5 (CC2), R7.1
- no-connect marks 0 -> 2

Commit message: Making progress
Parts:
- added D3: LED, LED_SMD:LED_1206_3216Metric_Pad1.42x1.75mm_HandSolder, symbol Device:LED
- added R17: 1k, Resistor_SMD:R_01005_0402Metric_Pad0.57x0.30mm_HandSolder, symbol Device:R_US
- C1: footprint Capacitor_SMD:C_1206_3216Metric_Pad1.33x1.80mm_HandSolder -> Capacitor_SMD:C_01005_0402Metric_Pad0.57x0.30mm_HandSolder
- C2, C3: footprint LED_SMD:LED_Kingbright_APFA3010_3x1.5mm_Horizontal -> Capacitor_SMD:C_01005_0402Metric_Pad0.57x0.30mm_HandSolder
- R16, R3, R4, R7: footprint Resistor_SMD:R_1206_3216Metric_Pad1.30x1.75mm_HandSolder -> Resistor_SMD:R_01005_0402Metric_Pad0.57x0.30mm_HandSolder
Connections:
- net GND: now also D3.1 (K)
- net VBUS: now also R17.2
- new net: D3.2 (A), R17.1

Commit message: making progress
Parts:
- C1, C2, C3: footprint Capacitor_SMD:C_01005_0402Metric_Pad0.57x0.30mm_HandSolder -> Capacitor_SMD:C_0201_0603Metric_Pad0.64x0.40mm_HandSolder
- R16, R17, R3, R4, R7: footprint Resistor_SMD:R_01005_0402Metric_Pad0.57x0.30mm_HandSolder -> Resistor_SMD:R_0201_0603Metric_Pad0.64x0.40mm_HandSolder
Changed lines of the file:
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@@
 			)
 		)
-		(property "Footprint" "Resistor_SMD:R_01005_0402Metric_Pad0.57x0.30mm_HandSolder"
+		(property "Footprint" "Resistor_SMD:R_0201_0603Metric_Pad0.64x0.40mm_HandSolder"
 			(at 91.694 163.576 90)
 			(hide yes)
@@
 			)
 		)
-		(property "Footprint" "Capacitor_SMD:C_01005_0402Metric_Pad0.57x0.30mm_HandSolder"
+		(property "Footprint" "Capacitor_SMD:C_0201_0603Metric_Pad0.64x0.40mm_HandSolder"
 			(at 179.07 80.01 0)
 			(hide yes)
@@
 			)
 		)
-		(property "Footprint" "Resistor_SMD:R_01005_0402Metric_Pad0.57x0.30mm_HandSolder"
+		(property "Footprint" "Resistor_SMD:R_0201_0603Metric_Pad0.64x0.40mm_HandSolder"
 			(at 85.344 86.614 90)
 			(hide yes)
@@
 			)
 		)
-		(property "Footprint" "Capacitor_SMD:C_01005_0402Metric_Pad0.57x0.30mm_HandSolder"
+		(property "Footprint" "Capacitor_SMD:C_0201_0603Metric_Pad0.64x0.40mm_HandSolder"
 			(at 248.92 80.01 0)
 			(hide yes)
@@
 			)
 		)
-		(property "Footprint" "Resistor_SMD:R_01005_0402Metric_Pad0.57x0.30mm_HandSolder"
+		(property "Footprint" "Resistor_SMD:R_0201_0603Metric_Pad0.64x0.40mm_HandSolder"
 			(at 131.064 67.056 90)
 			(hide yes)
@@
 			)
 		)
-		(property "Footprint" "Capacitor_SMD:C_01005_0402Metric_Pad0.57x0.30mm_HandSolder"
+		(property "Footprint" "Capacitor_SMD:C_0201_0603Metric_Pad0.64x0.40mm_HandSolder"
 			(at 129.54 171.45 0)
 			(hide yes)
@@
 			)
 		)
-		(property "Footprint" "Resistor_SMD:R_01005_0402Metric_Pad0.57x0.30mm_HandSolder"
+		(property "Footprint" "Resistor_SMD:R_0201_0603Metric_Pad0.64x0.40mm_HandSolder"
 			(at 85.344 94.234 90)
 			(hide yes)
@@
 			)
 		)
-		(property "Footprint" "Resistor_SMD:R_01005_0402Metric_Pad0.57x0.30mm_HandSolder"
+		(property "Footprint" "Resistor_SMD:R_0201_0603Metric_Pad0.64x0.40mm_HandSolder"
 			(at 91.694 180.086 90)
 			(hide yes)
@@
 		)
 	)
-	(embedded_fonts no)
 )

Commit message: Working
Connections:
- net D+: now also J2.B6 (DP2); no longer J2.A7 (DN1)
- net D-: now also J2.A7 (DN1); no longer J2.B6 (DP2)
Changed lines of the file:
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@@
-	)
-	(junction
-		(at 78.74 82.55)
-		(diameter 0)
-		(color 0 0 0 0)
 	)
 	(junction
@@
 	)
 	(junction
-		(at 78.74 74.93)
+		(at 80.01 105.41)
 		(diameter 0)
 		(color 0 0 0 0)
 	)
 	(junction
-		(at 80.01 105.41)
+		(at 77.47 80.01)
 		(diameter 0)
 		(color 0 0 0 0)
@@
 		(color 0 0 0 0)
 	)
+	(junction
+		(at 80.01 74.93)
+		(diameter 0)
+		(color 0 0 0 0)
+	)
 	(no_connect
 		(at 74.93 90.17)
@@
 	(wire
 		(pts
-			(xy 78.74 74.93) (xy 83.82 74.93)
+			(xy 74.93 80.01) (xy 77.47 80.01)
 		)
 		(stroke
@@
 	(wire
 		(pts
+			(xy 74.93 72.39) (xy 77.47 72.39)
+		)
+		(stroke
+			(width 0)
+			(type default)
+		)
+	)
+	(wire
+		(pts
 			(xy 85.09 168.91) (xy 92.71 168.91)
 		)
@@
 	(wire
 		(pts
-			(xy 74.93 74.93) (xy 78.74 74.93)
-		)
-		(stroke
-			(width 0)
-			(type default)
-		)
-	)
-	(wire
-		(pts
 			(xy 74.93 115.57) (xy 80.01 115.57)
 		)
@@
 	(wire
 		(pts
+			(xy 74.93 74.93) (xy 80.01 74.93)
+		)
+		(stroke
+			(width 0)
+			(type default)
+		)
+	)
+	(wire
+		(pts
 			(xy 191.77 82.55) (xy 198.12 82.55)
 		)
@@
 	(wire
 		(pts
-			(xy 78.74 72.39) (xy 78.74 74.93)
-		)
-		(stroke
-			(width 0)
-			(type default)
-		)
-	)
-	(wire
-		(pts
 			(xy 179.07 82.55) (xy 179.07 87.63)
 		)
@@
 	(wire
 		(pts
-			(xy 74.93 82.55) (xy 78.74 82.55)
-		)
-		(stroke
-			(width 0)
-			(type default)
-		)
-	)
-	(wire
-		(pts
 			(xy 248.92 74.93) (xy 248.92 71.12)
 		)
@@
 	(wire
 		(pts
-			(xy 78.74 82.55) (xy 83.82 82.55)
+			(xy 80.01 82.55) (xy 80.01 74.93)
+		)
+		(stroke
+			(width 0)
+			(type default)
+		)
+	)
+	(wire
+		(pts
+			(xy 77.47 80.01) (xy 83.82 80.01)
 		)
 		(stroke
@@
 	(wire
 		(pts
-			(xy 74.93 80.01) (xy 78.74 80.01)
-		)
-		(stroke
-			(width 0)
-			(type default)
-		)
-	)
-	(wire
-		(pts
 			(xy 92.71 184.15) (xy 92.71 187.96)
 		)
@@
 	(wire
 		(pts
-			(xy 78.74 80.01) (xy 78.74 82.55)
-		)
-		(stroke
-			(width 0)
-			(type default)
-		)
-	)
-	(wire
-		(pts
 			(xy 74.93 113.03) (xy 80.01 113.03)
 		)
@@
 	(wire
 		(pts
+			(xy 80.01 74.93) (xy 83.82 74.93)
+		)
+		(stroke
+			(width 0)
+			(type default)
+		)
+	)
+	(wire
+		(pts
 			(xy 88.9 87.63) (xy 93.98 87.63)
 		)
@@
 	(wire
 		(pts
+			(xy 74.93 82.55) (xy 80.01 82.55)
+		)
+		(stroke
+			(width 0)
+			(type default)
+		)
+	)
+	(wire
+		(pts
 			(xy 96.52 173.99) (xy 92.71 173.99)
 		)
@@
 	(wire
 		(pts
-			(xy 74.93 72.39) (xy 78.74 72.39)
-		)
-		(stroke
-			(width 0)
-			(type default)
-		)
-	)
-	(wire
-		(pts
 			(xy 92.71 187.96) (xy 85.09 187.96)
+		)
+		(stroke
+			(width 0)
+			(type default)
+		)
+	)
+	(wire
+		(pts
+			(xy 77.47 72.39) (xy 77.47 80.01)
 		)
 		(stroke
@@
 	(global_label "D-"
 		(shape input)
-		(at 83.82 82.55 0)
+		(at 83.82 80.01 0)
 		(fields_autoplaced yes)
 		(effects
@@
 		)
 		(property "Intersheetrefs" "${INTERSHEET_REFS}"
-			(at 89.6476 82.55 0)
+			(at 89.6476 80.01 0)
 			(hide yes)
 			(show_name no)
@@
 		)
 	)
-	(embedded_fonts no)
 )

Commit message: Working
Parts:
- D3: footprint LED_SMD:LED_1206_3216Metric_Pad1.42x1.75mm_HandSolder -> LED_SMD:LED_0603_1608Metric_Pad1.05x0.95mm_HandSolder
Changed lines of the file:
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@@
 			)
 		)
-		(property "Footprint" "LED_SMD:LED_1206_3216Metric_Pad1.42x1.75mm_HandSolder"
+		(property "Footprint" "LED_SMD:LED_0603_1608Metric_Pad1.05x0.95mm_HandSolder"
 			(at 132.08 78.74 0)
 			(hide yes)
@@
 		)
 	)
+	(embedded_fonts no)
 )
